File: kicad/ckt-soundplay-test/ckt-soundplay-test.kicad_sch (KiCad schematic)
At the start: 26 parts, among them J1 Screw_Terminal_01x02, J2 Screw_Terminal_01x02, J3 Screw_Terminal_01x02, J4 Screw_Terminal_01x02, J8 Screw_Terminal_01x02, J9 Conn_01x05, SW1 FSM4JSMATR, SW2 FSM4JSMATR, SW3 FSM4JSMATR, SW4 FSM4JSMATR, SW5 FSM4JSMATR, SW6 FSM4JSMATR

Commit message: Added holes for test points and rewired slightly
Parts:
- added TP1, TP2, TP3, TP4, TP5, TP6: TestPoint, Connector_PinHeader_2.54mm:PinHeader_1x01_P2.54mm_Vertical, symbol Connector:TestPoint
Connections:
- net GND: now also J4.2 (Pin_2), J8.2 (Pin_2), JP1.2 (Pin_2), JP2.1 (Pin_1), SW1.1, SW1.2, SW2.3, SW2.4, SW3.3, SW3.4, SW4.3, SW4.4, SW5.3, SW5.4, SW6.3, SW6.4, TP6.1
- net VPWR: now also TP5.1
- net at J4.1 (Pin_1), JMETER1.1 (Pin_1), SW3.1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: now also TP1.1
- net at J4.3 (Pin_3), SW4.1, SW4.2: now also TP2.1
- net at J8.1 (Pin_1), SW5.1, SW5.2: now also TP3.1
- net at J8.3 (Pin_3), SW6.1, SW6.2: now also TP4.1
Other:
- moved on the sheet: J4, J8
